Commit message: Checkpoint calibration and teaching workflows; improve visual teach UI and depth geometry

File: src/DOBOT_6Axis_ROS2_V4/cra_description/urdf/cr10_robot.xacro (robot description, xacro)
@@ -396,103 +396,3 @@
       velocity="100" />
   </joint>
-<gazebo reference="base_link">
-        <gravity>false</gravity>
-        <selfCollide>true</selfCollide>
-    </gazebo>
-    <gazebo reference="Link1">
-        <gravity>false</gravity>
-        <selfCollide>true</selfCollide>
-    </gazebo>
-    <gazebo reference="Link2">
-        <gravity>false</gravity>
-        <selfCollide>true</selfCollide>
-    </gazebo>
-    <gazebo reference="Link3">
-        <gravity>false</gravity>
-        <selfCollide>true</selfCollide>
-    </gazebo>
-    <gazebo reference="Link4">
-        <gravity>false</gravity>
-        <selfCollide>true</selfCollide>
-    </gazebo>
-    <gazebo reference="Link5">
-        <gravity>false</gravity>
-        <selfCollide>true</selfCollide>
-    </gazebo>
-    <gazebo reference="Link6">
-        <gravity>false</gravity>
-        <selfCollide>true</selfCollide>
-    </gazebo>
-    <!-- 在运行demo.launch.py时，需要注释这个ros2_control节点，因为它使用了xxx.ros2_control.xacro来生成了ros2_control节点-->
-    <ros2_control name="GazeboSystem" type="system">
-        <hardware>
-            <plugin>gazebo_ros2_control/GazeboSystem</plugin>
-        </hardware>
-        <joint name="joint1">
-            <command_interface name="position">
-                <param name="min">-1</param>
-                <param name="max">1</param>
-            </command_interface>
-            <state_interface name="position">
-                <param name="initial_value">0.0</param>
-            </state_interface>
-            <state_interface name="velocity"/>
-        </joint>
-        <joint name="joint2">
-            <command_interface name="position">
-                <param name="min">-1</param>
-                <param name="max">1</param>
-            </command_interface>
-            <state_interface name="position">
-                <param name="initial_value">0.0</param>
-            </state_interface>
-            <state_interface name="velocity"/>
-        </joint>
-        <joint name="joint3">
-            <command_interface name="position">
-                <param name="min">-1</param>
-                <param name="max">1</param>
-            </command_interface>
-            <state_interface name="position">
-                <param name="initial_value">0.0</param>
-            </state_interface>
-            <state_interface name="velocity"/>
-        </joint>
-        <joint name="joint4">
-            <command_interface name="position">
-                <param name="min">-1</param>
-                <param name="max">1</param>
-            </command_interface>
-            <state_interface name="position">
-                <param name="initial_value">0.0</param>
-            </state_interface>
-            <state_interface name="velocity"/>
-        </joint>
-        <joint name="joint5">
-            <command_interface name="position">
-                <param name="min">-1</param>
-                <param name="max">1</param>
-            </command_interface>
-            <state_interface name="position">
-                <param name="initial_value">0.0</param>
-            </state_interface>
-            <state_interface name="velocity"/>
-        </joint>
-        <joint name="joint6">
-            <command_interface name="position">
-                <param name="min">-1</param>
-                <param name="max">1</param>
-            </command_interface>
-            <state_interface name="position">
-                <param name="initial_value">0.0</param>
-            </state_interface>
-            <state_interface name="velocity"/>
-        </joint>
-    </ros2_control>
-    <gazebo>
-        <plugin filename="libgazebo_ros2_control.so" name="gazebo_ros2_control">
-            <parameters>$(find cr10_moveit)/config/ros2_controllers.yaml</parameters>
-            <robot_param_node>robot_state_publisher</robot_param_node>
-        </plugin>
-    </gazebo>
 </robot>
